File: numpad-test.kicad_pcb (KiCad board)
At the start: 2 copper layers, 100 x 100 mm, 78 parts, among them J1 Conn_01x03, J2 Conn_01x03, J3 Conn_OLED, J4 USB_C_Receptacle_USB2.0, SW1 SW_SPDT, SW10 SW_Push_45deg, SW11 SW_Push_45deg, SW12 SW_Push_45deg, SW13 SW_Push_45deg, SW14 SW_Push_45deg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

Commit message: <chore> remove anime silkscreen & gerber
Parts:
- removed G*** (x6): LOGO, LOGO
- moved ? 3.12 mm to (79.7, 50.5)
